File: KiCad/FrontPanel/FrontPanel.kicad_pcb (KiCad board)
At the start: 2 copper layers, 258.1 x 122.9 mm, 125 parts, among them J1 TO_FP, Q1 2N7002, Q2 2N7002, Q3 2N7002, Q4 2N7002, Q5 2N7002, SW1 SW_Push, SW10 SW_Push, SW11 SW_Push, SW12 SW_Push, SW13 SW_Push, SW14 SW_Push, SW15 SW_Push, SW16 SW_Push, SW17 SW_Push, SW18 SW_Push, SW19 SW_Push, SW2 SW_Push, SW20 SW_Push, SW3 SW_Push, SW4 SW_Push, SW5 SW_Push, SW6 SW_Push, SW7 SW_Push, SW8 SW_Push, SW9 SW_Push, U1 74HC244, U10 SM420561N, U11 SM420561N, U12 SM420561N, U13 SM420561N, U14 SM420561N, U15 SM420561N, U16 SM420561N, U17 SM420561N, U18 SM420561N, U19 SM420561N, U2 74HCT138, U20 SM420561N, U21 SM420561N, U22 NE555D, U3 74HCT138, U4 74HC244, U5 74HC244, U6 SM420561N, U7 SM420561N, U8 SM420561N, U9 SM420561N

Commit message: Prepare for bring-up
Parts:
- removed the ? at (75.2, 43.2)
- removed the ? at (271.3, 31.5)
- removed the ? at (17.3, 31.5)
- removed the ? at (136.1, 98.0)
- removed the ? at (271.3, 150.4)
- removed the ? at (17.3, 150.4)
- removed the ? at (236.7, 75.2)
- added ?: , , F.Cu at (270.8, 32.0)
- added ?: , , F.Cu at (270.8, 149.9)
- added ?: , , F.Cu at (17.8, 149.9)
- added ?: , , F.Cu at (136.7, 94.0)
- added ?: , , F.Cu at (234.2, 85.3)
- added ?: , , F.Cu at (17.8, 32.0)
Routing:
- net SEG_R2_C: track 0.00 -> 328.2 mm, vias 0 -> 2
- net SEG_R2_E: track 0.00 -> 323.8 mm, vias 0 -> 7
- net SEG_R2_D: track 0.00 -> 321.7 mm, vias 0 -> 1
- net SEG_R2_G: track 0.00 -> 312.7 mm, vias 0 -> 1
- net SEG_R2_A: track 0.00 -> 310.8 mm, vias 0 -> 2
- net SEG_R2_F: track 0.00 -> 307.1 mm, vias 0 -> 3
- net SEG_R2_DP: track 0.00 -> 306.1 mm, vias 0 -> 1
- net SEG_R2_B: track 0.00 -> 304.2 mm, vias 0 -> 2
- net SEG_R1_E: track 0.00 -> 297.7 mm, vias 0 -> 5
- net SIGN_R2: track 0.00 -> 295.8 mm, vias 0 -> 1
- net SEG_R1_C: track 0.00 -> 294.8 mm, vias 0 -> 2
- net SEG_R1_A: track 0.00 -> 286.4 mm, vias 0 -> 1
- net SEG_R1_D: track 0.00 -> 285.6 mm, vias 0 -> 6
- net SEG_R1_F: track 0.00 -> 278.5 mm, vias 0 -> 2
- net SEG_R1_G: track 0.00 -> 271.5 mm, vias 0 -> 1
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- added copper zone on F.Cu, net +5V
- added copper zone on B.Cu, net GND
Other:
- board text added: "LVDC Front Panel 0111 rev. 2025-04-24"
