File: KiCad/FrontPanel/FrontPanel.kicad_sch (KiCad schematic)
At the start: 118 parts, among them J1 TO_FP, Q1 2N7002, Q2 2N7002, Q3 2N7002, Q4 2N7002, Q5 2N7002, SW1 SW_Push, SW10 SW_Push, SW11 SW_Push, SW12 SW_Push, SW13 SW_Push, SW14 SW_Push, SW15 SW_Push, SW16 SW_Push, SW17 SW_Push, SW18 SW_Push, SW19 SW_Push, SW2 SW_Push, SW20 SW_Push, SW3 SW_Push, SW4 SW_Push, SW5 SW_Push, SW6 SW_Push, SW7 SW_Push, SW8 SW_Push, SW9 SW_Push, U1 74HC244, U10 SM420561N, U11 SM420561N, U12 SM420561N, U13 SM420561N, U14 SM420561N, U15 SM420561N, U16 SM420561N, U17 SM420561N, U18 SM420561N, U19 SM420561N, U2 74HCT138, U20 SM420561N, U21 SM420561N, U22 NE555D, U3 74HCT138, U4 74HC244, U5 74HC244, U6 SM420561N, U7 SM420561N, U8 SM420561N, U9 SM420561N

Commit message: Prepare for bring-up
Connections:
- no-connect marks 5 -> 7
Changed lines of the file:
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@@
+	)
+	(no_connect
+		(at 55.88 55.88)
 	)
 	(no_connect
@@
 	)
 	(no_connect
+		(at 55.88 53.34)
+	)
+	(no_connect
