File: KiCad/GPIO/GPIO.kicad_pcb (KiCad board)
At the start: 4 copper layers, 209.6 x 108.5 mm, 112 parts, among them J1 JTAG, J10 Conn_01x01, J11 TO_FP, J12 Conn_01x04, J13 Conn_01x08, J14 Conn_01x08, J15 RADIO_MODULE, J2 TO_BACKPLANE, J3 Conn_01x01, J4 Conn_01x01, J5 Conn_01x01, J6 AUDIO_OUT, J7 Conn_01x04, J8 Conn_01x04, J9 RADIO_MODULE, U1 EPM240T100, U10 SN74ALVC164245DGG, U11 SN74LV1T34DCK, U12 SN74LV1T34DCK, U13 SN74LV1T34DCK, U14 SN74LV1T34DCK, U15 74HC74, U16 gfmpw1-multi, U17 DAC7611, U18 DAC7611, U19 LM358, U2 MCP1319MT-29LE-OT, U20 SN74LV1T34DCK, U21 SN74LV1T34DCK, U22 SN74LV1T34DCK, U23 HT12D, U24 SN74LV1T34DCK, U25 74HCT244, U26 74HCT244, U27 SN74LV1T34DCK, U28 SN74LV1T34DCK, U29 74HC32, U3 W25Q32FVSS, U30 74HC574, U31 74AHC1G86, U32 HT12E, U33 SN74LV1T34DCK, U34 SN74LV1T34DCK, U35 SN74LV1T34DCK, U4 AMS1117-3.3, U5 74HC574, U6 74HCT244, U7 74HCT74, U8 SN74LV1T34DCK, U9 SN74LV1T34DCK, X1 CXO_DIP8

Commit message: Prepare for bring-up
Parts:
- added J16: Conn_01x04, Connector_PinHeader_2.54mm:PinHeader_1x04_P2.54mm_Vertical, F.Cu at (113.3, 67.1)
Connections:
- U1 pad 90: unconnected-(U1-IO2_90-Pad90) -> Net-(J16-Pin_1)
- U1 pad 91: unconnected-(U1-IO2_91-Pad91) -> Net-(J16-Pin_2)
Routing:
- net Net-(J16-Pin_2): track 0.00 -> 27.8 mm, vias 0 -> 2
- net Net-(J16-Pin_1): track 0.00 -> 27.4 mm, vias 0 -> 2
- net ~{SID_CE}: track 143.8 -> 144.7 mm
- net GND: track 186.1 -> 186.7 mm
Other:
- board text added: "+5V"
- board text added: "GND"
- board text added: "SCL"
- board text added: "SDA"
