File: KiCad/ALU/ALU.kicad_sch (KiCad schematic)
At the start: 33 parts, among them J1 ACCUMULATOR, J2 TO_BACKPLANE, J3 FROM_CTRL, U1 74HCT04, U16 74LS181, U17 74LS181, U18 74LS181, U19 74LS181, U20 74LS181, U21 74LS181, U22 74LS181, U23 74HCT08, U24 74HCT08, U25 74HCT32

Commit message: Update schematics with fixes.
Connections:
- no-connect marks 19 -> 22
Changed lines of the file:
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@@
 (kicad_sch
-	(version 20231120)
+	(version 20250114)
 	(generator "eeschema")
-	(generator_version "8.0")
+	(generator_version "9.0")
 	(paper "A3")
 	(junction
@@
 	)
 	(no_connect
+		(at 158.75 200.66)
+	)
+	(no_connect
 		(at 219.71 203.2)
 	)
@@
 	)
 	(no_connect
+		(at 158.75 195.58)
+	)
+	(no_connect
 		(at 190.5 266.7)
 	)
@@
 	)
 	(no_connect
+		(at 158.75 203.2)
+	)
+	(no_connect
 		(at 158.75 63.5)
 	)
@@
 		(at 332.74 105.41)
 		(size 41.91 20.32)
+		(exclude_from_sim no)
+		(in_bom yes)
+		(on_board yes)
+		(dnp no)
 		(fields_autoplaced yes)
 		(stroke
@@
 		(at 81.28 257.81)
 		(size 29.21 13.97)
+		(exclude_from_sim no)
+		(in_bom yes)
+		(on_board yes)
+		(dnp no)
 		(fields_autoplaced yes)
 		(stroke
@@
 		(at 77.47 90.17)
 		(size 15.24 7.62)
+		(exclude_from_sim no)
+		(in_bom yes)
+		(on_board yes)
+		(dnp no)
 		(fields_autoplaced yes)
 		(stroke
@@
 		)
 	)
+	(embedded_fonts no)
 )
