File: KiCad/Control/Control.kicad_pcb (KiCad board)
At the start: 4 copper layers, 209.5 x 108.5 mm, 79 parts, among them J1 TO_BACKPLANE, J2 TO_ALU, J3 TO_MEMORY, J4 TO_REGISTERS, J5 TO_MULDIV, J6 Conn_01x01, J7 Conn_01x01, J8 Conn_01x01, U1 74HC574, U10 74HCT32, U11 74HCT08, U12 28C16, U13 28C16, U14 74HCT163, U15 74HCT00, U16 74HCT32, U17 74HCT04, U18 74HCT74, U19 74HCT74, U2 74HCT04, U20 74HCT157, U21 74HCT08, U22 74HCT32, U23 74HCT04, U24 74HCT08, U25 74HCT08, U26 74HCT74, U27 74HCT74, U28 74HCT08, U29 74HCT32, U3 74HCT157, U30 74HCT08, U31 74HC85, U32 74HC85, U33 74HC74, U34 74HC688, U35 74HC00, U36 74HCT157, U37 74HCT157, U38 74HCT157, U39 74HCT157, U4 74HCT157, U5 74HCT157, U6 74HCT157, U7 74HC574, U8 74HCT157, U9 74HCT08

Commit message: Update schematics with fixes.
Parts:
- added U40: 74HC74, Package_SO:SO-14_3.9x8.65mm_P1.27mm, F.Cu at (-15.0, 65.6)
- added U41: 74HC02, Package_SO:SO-14_3.9x8.65mm_P1.27mm, F.Cu at (-6.52, 65.6)
Connections:
- J4 pad 10: H_CYC_1 -> GND
- U16 pad 5: I1 -> I2
- U17 pad 3: I2 -> I1
- U2 pad 1: Net-(U18A-D) -> Net-(U2-Pad1)
- U29 pad 10: GND -> INT_INHIBIT2
- U29 pad 8: unconnected-(U29-Pad8) -> Net-(U2-Pad1)
- U29 pad 9: RST -> Net-(U18A-D)
- U34 pad 1: GND -> ~{IOR}
- U34 pad 19: Net-(U34-P=R) -> ICLR
- U35 pad 2: Net-(U34-P=R) -> +5V
- U35 pad 3: ICLR -> unconnected-(U35-Pad3)
Routing:
- net CLK: track 459.1 -> 0.00 mm, vias 9 -> 0
- net ~{RST}: track 393.7 -> 0.00 mm, vias 4 -> 0
- net IS_EXM_I: track 342.1 -> 0.00 mm, vias 8 -> 0
- net I2: track 293.8 -> 0.00 mm, vias 7 -> 0
- net I1: track 289.7 -> 0.00 mm, vias 5 -> 0
- net I3: track 286.1 -> 0.00 mm, vias 4 -> 0
- net I0: track 265.8 -> 0.00 mm, vias 5 -> 0
- net FETCH_CYC: track 259.0 -> 0.00 mm, vias 7 -> 0
- net I4: track 256.3 -> 0.00 mm, vias 4 -> 0
- net I12: track 244.5 -> 0.00 mm, vias 6 -> 0
- net irupt: track 242.5 -> 0.00 mm, vias 3 -> 0
- net H_CYC_1: track 230.3 -> 0.00 mm, vias 5 -> 0
- net RST: track 227.4 -> 0.00 mm, vias 6 -> 0
- net MEM_RD: track 198.5 -> 0.00 mm, vias 1 -> 0
- net I7: track 192.9 -> 0.00 mm, vias 4 -> 0
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