File: KiCad/Control/IOCTRL.kicad_sch (KiCad schematic)
At the start: 2 parts, among them U34 74HC688, U35 74HC00

Commit message: Update schematics with fixes.
Connections:
- net +5V: now also U35.2
- net GND: no longer U34.1 (G)
- net ICLR: now also U34.19 (P=R); no longer U35.3
- net ~{IOR}: now also U34.1 (G)
- no-connect marks 0 -> 1
Other:
- note added: "Uh-oh, this does not check that its an IO op A regular memory access will trigger ICLR!"
- moved on the sheet: U35A
Changed lines of the file:
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@@
 	(generator_version "9.0")
 	(paper "A4")
+	(text "Uh-oh, this does not check that its an IO op\nA regular memory access will trigger ICLR!"
+		(exclude_from_sim no)
+		(at 70.612 47.498 0)
+		(effects
+			(font
+				(size 1.27 1.27)
+			)
+		)
+	)
+	(junction
+		(at 102.87 34.29)
+		(diameter 0)
+		(color 0 0 0 0)
+	)
 	(junction
 		(at 102.87 100.33)
@@
 		(color 0 0 0 0)
 	)
+	(no_connect
+		(at 119.38 36.83)
+	)
 	(wire
 		(pts
@@
 	(wire
 		(pts
-			(xy 119.38 86.36) (xy 119.38 91.44)
+			(xy 102.87 39.37) (xy 102.87 34.29)
 		)
 		(stroke
@@
 	(wire
 		(pts
-			(xy 95.25 58.42) (xy 95.25 62.23)
+			(xy 104.14 39.37) (xy 102.87 39.37)
 		)
 		(stroke
@@
 	(wire
 		(pts
-			(xy 95.25 62.23) (xy 96.52 62.23)
+			(xy 119.38 86.36) (xy 119.38 91.44)
 		)
 		(stroke
@@
 	(wire
 		(pts
-			(xy 134.62 78.74) (xy 139.7 78.74)
+			(xy 102.87 30.48) (xy 102.87 34.29)
 		)
 		(stroke
@@
 	(wire
 		(pts
-			(xy 97.79 100.33) (xy 100.33 100.33)
+			(xy 114.3 64.77) (xy 115.57 64.77)
 		)
 		(stroke
@@
 	(wire
 		(pts
-			(xy 118.11 102.87) (xy 118.11 96.52)
+			(xy 102.87 34.29) (xy 104.14 34.29)
 		)
 		(stroke
@@
 	(wire
 		(pts
-			(xy 85.09 67.31) (xy 96.52 67.31)
+			(xy 134.62 78.74) (xy 139.7 78.74)
 		)
 		(stroke
@@
 	(wire
 		(pts
-			(xy 119.38 81.28) (xy 119.38 86.36)
+			(xy 97.79 100.33) (xy 100.33 100.33)
 		)
 		(stroke
@@
 	(wire
 		(pts
-			(xy 100.33 76.2) (xy 100.33 100.33)
+			(xy 118.11 102.87) (xy 118.11 96.52)
 		)
 		(stroke
@@
 	(wire
 		(pts
-			(xy 111.76 64.77) (xy 115.57 64.77)
+			(xy 119.38 81.28) (xy 119.38 86.36)
 		)
 		(stroke
@@
 	(wire
 		(pts
-			(xy 118.11 86.36) (xy 119.38 86.36)
+			(xy 100.33 76.2) (xy 100.33 100.33)
 		)
 		(stroke
@@
 	(wire
 		(pts
-			(xy 100.33 100.33) (xy 102.87 100.33)
+			(xy 118.11 86.36) (xy 119.38 86.36)
 		)
 		(stroke
@@
 	(wire
 		(pts
-			(xy 118.11 96.52) (xy 119.38 96.52)
+			(xy 100.33 100.33) (xy 102.87 100.33)
 		)
 		(stroke
@@
 	(wire
 		(pts
-			(xy 119.38 76.2) (xy 100.33 76.2)
+			(xy 118.11 96.52) (xy 119.38 96.52)
 		)
 		(stroke
@@
 	(wire
 		(pts
-			(xy 134.62 93.98) (xy 139.7 93.98)
+			(xy 119.38 76.2) (xy 100.33 76.2)
 		)
 		(stroke
@@
 		)
 	)
+	(wire
+		(pts
+			(xy 85.09 67.31) (xy 114.3 67.31)
+		)
+		(stroke
+			(width 0)
+			(type default)
+		)
+	)
+	(wire
+		(pts
+			(xy 134.62 93.98) (xy 139.7 93.98)
+		)
+		(stroke
+			(width 0)
+			(type default)
+		)
+	)
+	(wire
+		(pts
+			(xy 114.3 67.31) (xy 114.3 64.77)
+		)
+		(stroke
+			(width 0)
+			(type default)
+		)
+	)
 	(global_label "I4"
 		(shape input)
@@
 				)
 				(justify left)
+				(hide yes)
+			)
+		)
+	)
+	(global_label "~{IOR}"
+		(shape input)
+		(at 59.69 113.03 180)
+		(fields_autoplaced yes)
+		(effects
+			(font
+				(size 1.27 1.27)
+			)
+			(justify right)
+		)
+		(property "Intersheetrefs" "${INTERSHEET_REFS}"
+			(at 53.4995 113.03 0)
+			(effects
+				(font
+					(size 1.27 1.27)
+				)
+				(justify right)
 				(hide yes)
 			)
@@
 	(symbol
 		(lib_id "74xx:74HC00")
-		(at 104.14 64.77 0)
+		(at 111.76 36.83 0)
 		(unit 1)
 		(exclude_from_sim no)
@@
 		(fields_autoplaced yes)
 		(property "Reference" "U35"
-			(at 104.1317 55.88 0)
+			(at 111.7517 27.94 0)
 			(effects
 				(font
@@
 		)
 		(property "Value" "74HC00"
-			(at 104.1317 58.42 0)
+			(at 111.7517 30.48 0)
 			(effects
 				(font
@@
 		)
 		(property "Footprint" "Package_SO:SO-14_3.9x8.65mm_P1.27mm"
-			(at 104.14 64.77 0)
+			(at 111.76 36.83 0)
 			(effects
 				(font
@@
 		)
 		(property "Datasheet" "http://www.ti.com/lit/gpn/sn74hc00"
-			(at 104.14 64.77 0)
+			(at 111.76 36.83 0)
 			(effects
 				(font
@@
 		)
 		(property "Description" "quad 2-input NAND gate"
-			(at 104.14 64.77 0)
+			(at 111.76 36.83 0)
 			(effects
 				(font
@@
 		)
 		(property "VerilogCode" "ttl_74hct00 U35(_1, _2, _3, _4, _5, _6, _9, _10, _8, _12, _13, _11);"
-			(at 104.14 64.77 0)
+			(at 111.76 36.83 0)
 			(effects
 				(font
@@
 	(symbol
 		(lib_id "power:+5V")
-		(at 95.25 58.42 0)
+		(at 102.87 30.48 0)
 		(unit 1)
 		(exclude_from_sim no)
@@
 		(fields_autoplaced yes)
 		(property "Reference" "#PWR0138"
-			(at 95.25 62.23 0)
+			(at 102.87 34.29 0)
 			(effects
 				(font
@@
 		)
 		(property "Value" "+5V"
-			(at 95.25 53.34 0)
+			(at 102.87 25.4 0)
 			(effects
 				(font
@@
 		)
 		(property "Footprint" ""
-			(at 95.25 58.42 0)
+			(at 102.87 30.48 0)
 			(effects
 				(font
@@
 		)
 		(property "Datasheet" ""
-			(at 95.25 58.42 0)
+			(at 102.87 30.48 0)
 			(effects
 				(font
@@
 		)
 		(property "Description" "Power symbol creates a global label with name \"+5V\""
-			(at 95.25 58.42 0)
+			(at 102.87 30.48 0)
 			(effects
 				(font
@@
 					(unit 1)
 				)
-			)
-		)
-	)
-	(symbol
-		(lib_id "power:GND")
-		(at 59.69 113.03 270)
-		(unit 1)
-		(exclude_from_sim no)
-		(in_bom yes)
-		(on_board yes)
-		(dnp no)
-		(fields_autoplaced yes)
-		(property "Reference" "#PWR0135"
-			(at 53.34 113.03 0)
-			(effects
-				(font
-					(size 1.27 1.27)
-				)
-				(hide yes)
-			)
-		)
-		(property "Value" "GND"
-			(at 55.88 113.0299 90)
-			(effects
-				(font
-					(size 1.27 1.27)
-				)
-				(justify right)
-			)
-		)
-		(property "Footprint" ""
-			(at 59.69 113.03 0)
-			(effects
-				(font
-					(size 1.27 1.27)
-				)
-				(hide yes)
-			)
-		)
-		(property "Datasheet" ""
-			(at 59.69 113.03 0)
-			(effects
-				(font
-					(size 1.27 1.27)
-				)
-				(hide yes)
-			)
-		)
-		(property "Description" "Power symbol creates a global label with name \"GND\" , ground"
-			(at 59.69 113.03 0)
-			(effects
-				(font
-					(size 1.27 1.27)
-				)
-				(hide yes)
-			)
-		)
-		(pin "1"
-		)
-		(instances
-			(project "Control"
-				(path "/d9911e88-3002-43fe-906c-efbbcc56ef85/50940dae-6cbd-4a36-a566-8240c00b6567"
-					(reference "#PWR0135")
-					(unit 1)
-				)
