File: KiCad/Control/MEMCTRL.kicad_sch (KiCad schematic)
At the start: 11 parts, among them U10 74HCT32, U18 74HCT74, U19 74HCT74, U2 74HCT04, U20 74HCT157, U21 74HCT08, U22 74HCT32

Commit message: Update schematics with fixes.
Parts:
- added U29: 74HCT32, Package_SO:SO-14_3.9x8.65mm_P1.27mm, symbol 74xx:74LS32
Connections:
- net at U10.8, U18.2 (D): now also U29.9; no longer U2.1
- new net: U2.1, U29.8
- new net INT_INHIBIT2: U29.10
